Commit message: Add ros2_control + gz_ros2_control integration, working diff-drive sim in Gazebo

File: rover_description/urdf/rover.urdf.xacro (robot description, xacro)
@@ -138,17 +138,22 @@
     <material>Gazebo/DarkGrey</material>
   </gazebo>
-<!-- ===================== Gazebo: differential drive plugin ===================== -->
+  <ros2_control name="RoverSystem" type="system">
+    <hardware>
+      <plugin>gz_ros2_control/GazeboSimSystem</plugin>
+    </hardware>
+    <joint name="left_wheel_joint">
+      <command_interface name="velocity"/>
+      <state_interface name="velocity"/>
+      <state_interface name="position"/>
+    </joint>
+    <joint name="right_wheel_joint">
+      <command_interface name="velocity"/>
+      <state_interface name="velocity"/>
+      <state_interface name="position"/>
+    </joint>
+  </ros2_control>
   <gazebo>
-    <plugin filename="gz-sim-diff-drive-system" name="gz::sim::systems::DiffDrive">
-      <left_joint>left_wheel_joint</left_joint>
-      <right_joint>right_wheel_joint</right_joint>
-      <wheel_separation>${wheel_separation}</wheel_separation>
-      <wheel_radius>${wheel_radius}</wheel_radius>
-      <max_linear_acceleration>1.0</max_linear_acceleration>
-      <topic>cmd_vel</topic>
-      <odom_topic>odom</odom_topic>
-      <frame_id>odom</frame_id>
-      <child_frame_id>base_footprint</child_frame_id>
-      <odom_publish_frequency>30</odom_publish_frequency>
+    <plugin filename="gz_ros2_control-system" name="gz_ros2_control::GazeboSimROS2ControlPlugin">
+      <parameters>$(find rover_description)/config/controllers.yaml</parameters>
     </plugin>
   </gazebo>

Commit message: Add LiDAR sensor, room.sdf world, slam_toolbox integration, and synthetic /scan workaround for WSL2 Gazebo rendering bug

File: rover_description/urdf/rover.urdf.xacro (robot description, xacro)
@@ -18,4 +18,7 @@
   <xacro:property name="mesh_scale" value="0.001 0.001 0.001"/>
   <xacro:property name="base_mesh_rpy" value = "1.5708 0 0"/>
+  <xacro:property name="lidar_offset_x" value="0.0"/>
+  <xacro:property name="lidar_offset_y" value="0.0"/>
+  <xacro:property name="lidar_offset_z" value="0.08"/>
   <link name="base_footprint"/>
   <joint name="base_joint" type="fixed">
@@ -125,4 +128,28 @@
     <origin xyz="${sensor_offset_x} 0 ${sensor_offset_z}" rpy="0 0 0"/>
   </joint>
+  <link name="lidar_link">
+    <visual>
+      <geometry>
+        <cylinder radius="0.02" length="0.03"/>
+      </geometry>
+      <material name="black">
+        <color rgba="0.1 0.1 0.1 1"/>
+      </material>
+    </visual>
+    <collision>
+      <geometry>
+        <cylinder radius="0.02" length="0.03"/>
+      </geometry>
+    </collision>
+    <inertial>
+      <mass value="0.05"/>
+      <inertia ixx="1e-5" ixy="0" ixz="0" iyy="1e-5" iyz="0" izz="1e-5"/>
+    </inertial>
+  </link>
+  <joint name="lidar_joint" type="fixed">
+    <parent link="base_link"/>
+    <child link="lidar_link"/>
+    <origin xyz="${lidar_offset_x} ${lidar_offset_y} ${lidar_offset_z}" rpy="0 0 0"/>
+  </joint>
 <!-- ===================== Gazebo materials ===================== -->
   <gazebo reference="base_link">
@@ -137,4 +164,28 @@
   <gazebo reference="caster_link">
     <material>Gazebo/DarkGrey</material>
+  </gazebo>
+  <gazebo reference="lidar_link">
+    <sensor name="lidar" type="lidar">
+      <pose>0 0 0 0 0 0</pose>
+      <topic>scan</topic>
+      <update_rate>10</update_rate>
+      <always_on>true</always_on>
+      <visualize>true</visualize>
+      <lidar>
+        <scan>
+          <horizontal>
+            <samples>360</samples>
+            <resolution>1</resolution>
+            <min_angle>-3.14159</min_angle>
+            <max_angle>3.14159</max_angle>
+          </horizontal>
+        </scan>
+        <range>
+          <min>0.12</min>
+          <max>10.0</max>
+          <resolution>0.01</resolution>
+        </range>
+      </lidar>
+    </sensor>
   </gazebo>
   <ros2_control name="RoverSystem" type="system">

Commit message: Add simulated IMU, ground-truth odometry source, and robot_localization EKF fusion; fix use_sim_time defaults on fake sensor publishers; add spin_test validation script

File: rover_description/urdf/rover.urdf.xacro (robot description, xacro)
@@ -147,4 +147,48 @@
     </inertial>
   </link>
+  <link name="imu_link">
+    <visual>
+    <geometry>
+      <box size="0.02 0.02 0.01"/>
+    </geometry>
+    <material name="green">
+      <color rgba="0 0.6 0 1"/>
+    </material>
+  </visual>
+  <collision>
+    <geometry>
+      <box size="0.02 0.02 0.01"/>
+    </geometry>
+  </collision>
+  <inertial>
+    <mass value="0.01"/>
+    <inertia ixx="1e-7" ixy="0" ixz="0" iyy="1e-7" iyz="0" izz="1e-7"/>
+  </inertial>
+</link>
+<joint name="imu_joint" type="fixed">
+  <parent link="base_link"/>
+  <child link="imu_link"/>
+  <origin xyz="0 0 0.04" rpy="0 0 0"/>
+</joint>
+<gazebo reference="imu_link">
+  <sensor name="imu_sensor" type="imu">
+    <always_on>true</always_on>
+    <update_rate>100</update_rate>
+    <visualize>false</visualize>
+    <topic>imu</topic>
+    <imu>
+      <angular_velocity>
+        <x><noise type="gaussian"><mean>0.0</mean><stddev>0.0009</stddev></noise></x>
+        <y><noise type="gaussian"><mean>0.0</mean><stddev>0.0009</stddev></noise></y>
+        <z><noise type="gaussian"><mean>0.0</mean><stddev>0.0009</stddev></noise></z>
+      </angular_velocity>
+      <linear_acceleration>
+        <x><noise type="gaussian"><mean>0.0</mean><stddev>0.004</stddev></noise></x>
+        <y><noise type="gaussian"><mean>0.0</mean><stddev>0.004</stddev></noise></y>
+        <z><noise type="gaussian"><mean>0.0</mean><stddev>0.004</stddev></noise></z>
+      </linear_acceleration>
+    </imu>
+  </sensor>
+</gazebo>
   <joint name="lidar_joint" type="fixed">
     <parent link="base_link"/>
@@ -209,3 +253,12 @@
     </plugin>
   </gazebo>
+  <gazebo>
+    <plugin filename="gz-sim-odometry-publisher-system" name="gz::sim::systems::OdometryPublisher">
+      <odom_frame>ground_truth_odom</odom_frame>
+      <robot_base_frame>base_footprint</robot_base_frame>
+      <odom_topic>/model/rover/odometry_ground_truth</odom_topic>
+      <odom_publish_frequency>100</odom_publish_frequency>
+      <dimensions>2</dimensions>
+    </plugin>
+  </gazebo>
 </robot>

Commit message: Tiered chassis redesign: xacro rework, mesh updates, remove stale mesh files

File: rover_description/urdf/rover.urdf.xacro (robot description, xacro)
@@ -4,15 +4,23 @@
   <xacro:property name="base_length" value="0.300"/>
   <xacro:property name="base_width"  value="0.250"/>
-  <xacro:property name="base_thickness" value="0.005"/>
-  <xacro:property name="ground_clearance" value="0.025"/>
+  <xacro:property name="base_thickness" value="0.100"/>
+  <xacro:property name="base_height" value="${base_thickness}"/>
+  <xacro:property name="base_collision_z" value="${base_height/2}"/>
+  <xacro:property name="ground_clearance" value="0.0156"/>
+  <xacro:property name="caster_visual_rpy" value="-1.5708 0 0"/>
+  <xacro:property name="caster_ground_reach" value="0.0156"/>
+  <xacro:property name="caster_ball_radius" value="0.007"/>
   <xacro:property name="wheel_radius" value="0.0425"/>
   <xacro:property name="wheel_thickness" value="0.026"/>
-  <xacro:property name="wheel_separation" value="0.180"/>
-  <xacro:property name="wheel_axle_x" value="-0.085"/>
-  <xacro:property name="caster_offset_x_from_axle" value="0.210"/>
+  <xacro:property name="wheel_separation" value="0.235"/>
+  <xacro:property name="wheel_axle_x" value="0.050"/>
+  <xacro:property name="caster_offset_x_from_axle" value="-0.175"/>
   <xacro:property name="caster_x" value="${wheel_axle_x + caster_offset_x_from_axle}"/>
   <xacro:property name="sensor_offset_x" value="0.150"/>
   <xacro:property name="sensor_offset_z" value="0.0425"/>
-  <xacro:property name="base_link_z" value="${ground_clearance + base_thickness/2}"/>
+  <xacro:property name="base_link_z" value="${ground_clearance}"/>
+  <xacro:property name="base_visual_x" value="0.150"/>
+  <xacro:property name="base_visual_y" value="0.125"/>
+  <xacro:property name="base_visual_z" value="0.005"/>
   <xacro:property name="wheel_z" value="${wheel_radius - base_link_z}"/>
   <xacro:property name="mesh_scale" value="0.001 0.001 0.001"/>
@@ -20,5 +28,5 @@
   <xacro:property name="lidar_offset_x" value="0.0"/>
   <xacro:property name="lidar_offset_y" value="0.0"/>
-  <xacro:property name="lidar_offset_z" value="0.08"/>
+  <xacro:property name="lidar_offset_z" value="0.100"/>
   <link name="base_footprint"/>
   <joint name="base_joint" type="fixed">
@@ -29,5 +37,5 @@
   <link name="base_link">
     <visual>
-      <origin xyz="-0.150 0.125 0" rpy="${base_mesh_rpy}"/>
+      <origin xyz="${base_visual_x} ${base_visual_y} ${base_visual_z}" rpy="${base_mesh_rpy}"/>
       <geometry>
         <mesh filename="package://rover_description/meshes/base_plate.stl" scale="${mesh_scale}"/>
@@ -35,6 +43,7 @@
     </visual>
     <collision>
-      <geometry>
-        <box size="${base_length} ${base_width} ${base_thickness}"/>
+      <origin xyz="0 0 ${base_collision_z}" rpy="0 0 0"/>
+      <geometry>
+        <box size="${base_length} ${base_width} ${base_height}"/>
       </geometry>
     </collision>
@@ -46,7 +55,7 @@
   <link name="left_wheel_link">
     <visual>
-      <origin xyz="0.235 0.215 -0.024" rpy="1.5708 0 0"/>
-      <geometry>
-        <mesh filename="package://rover_description/meshes/wheel_left.stl" scale="${mesh_scale}"/>
+      <origin xyz="0 -0.013 0" rpy="0 0 1.5708"/>
+      <geometry>
+        <mesh filename="package://rover_description/meshes/wheel.stl" scale="${mesh_scale}"/>
       </geometry>
     </visual>
@@ -71,7 +80,7 @@
   <link name="right_wheel_link">
     <visual>
-      <origin xyz="0.235 0.035 -0.024" rpy="1.5708 0 0"/>
-      <geometry>
-        <mesh filename="package://rover_description/meshes/wheel_right.stl" scale="${mesh_scale}"/>
+      <origin xyz="0 -0.013 0" rpy="0 0 1.5708"/>
+      <geometry>
+        <mesh filename="package://rover_description/meshes/wheel.stl" scale="${mesh_scale}"/>
       </geometry>
     </visual>
@@ -96,18 +105,13 @@
   <link name="caster_link">
     <visual>
-    <origin xyz="0.025 0.125 0" rpy="1.5708 0 0"/>
-      <geometry>
-        <mesh filename="package://rover_description/meshes/caster_body.stl" scale="${mesh_scale}"/>
-      </geometry>
-    </visual>
-    <visual>
-    <origin xyz="0.025 0.125 0.001602" rpy="1.5708 0 0"/>
-      <geometry>
-        <mesh filename="package://rover_description/meshes/caster_ball.stl" scale="${mesh_scale}"/>
-      </geometry>
-    </visual>
-    <collision>
-      <geometry>
-        <sphere radius="0.010"/>
+      <origin xyz="0 0 0" rpy="${caster_visual_rpy}"/>
+      <geometry>
+        <mesh filename="package://rover_description/meshes/caster.stl" scale="${mesh_scale}"/>
+      </geometry>
+    </visual>
+    <collision>
+      <origin xyz="0 0 ${-caster_ground_reach + caster_ball_radius}" rpy="0 0 0"/>
+      <geometry>
+        <sphere radius="${caster_ball_radius}"/>
       </geometry>
     </collision>
@@ -169,5 +173,5 @@
   <parent link="base_link"/>
   <child link="imu_link"/>
-  <origin xyz="0 0 0.04" rpy="0 0 0"/>
+  <origin xyz="0 0 0.100" rpy="0 0 0"/>
 </joint>
 <gazebo reference="imu_link">
